File: Lora.kicad_pcb (KiCad board)
At the start: 4 copper layers, 27.1 x 70.5 mm, 50 parts, among them J1 USB_C_Receptacle_USB2.0_16P, SW1 BOOTSEL, SW2 RESET, U1 SX1262IMLTRT, U2 RP2040, U3 W25Q128JVS, U4 AP2112K-3.3, U5 PE4259, Y1 32mhz, Y2 12mhz

Commit message: dun x2
Parts:
- added G***: LOGO, foot:me, F.Cu at (120.3, 45.9)
- added G***: LOGO, foot:EU invert, B.Cu at (122.1, 46.6)
- added G***: LOGO, foot:Hazard, B.Cu at (139.7, 97.7)
- added G***: LOGO, foot:Ham big, B.Cu at (132.2, 68.7)
- added G***: LOGO, foot:EU, B.Cu at (141.0, 46.4)
- added G***: LOGO, foot:HCB, F.Cu at (140.3, 43.7)
- added G***: LOGO, foot:Warning, F.Cu at (140.7, 50.2)
- added G***: LOGO, foot:Me new, F.Cu at (123.2, 76.0)
- added G***: LOGO, foot:ham, F.Cu at (123.6, 88.9)
- added G***: LOGO, foot:Flame, B.Cu at (131.7, 97.7)
- added G***: LOGO, foot:EU invert, B.Cu at (141.0, 46.4)
- added G***: LOGO, foot:bomb, B.Cu at (123.7, 97.7)
- added REF**: MountingHole_2.2mm_M2, MountingHole:MountingHole_2.2mm_M2, F.Cu at (142.2, 38.9)
- added REF**: MountingHole_2.2mm_M2, MountingHole:MountingHole_2.2mm_M2, F.Cu at (121.0, 103.4)
- added REF**: MountingHole_2.2mm_M2, MountingHole:MountingHole_2.2mm_M2, F.Cu at (142.2, 103.5)
- added REF**: MountingHole_2.2mm_M2, MountingHole:MountingHole_2.2mm_M2, F.Cu at (121.0, 38.9)
- moved G*** 4.13 mm to (123.1, 98.6)
Other:
- board text added: "1GHz"
- board text added: "Boot"
- board text added: "Reset"

Commit message: Add files via upload
Parts:
- moved G*** 0.57 mm to (123.1, 99.2)
Changed lines of the file:
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@@
 	(footprint "foot:Orph letb smol"
 		(layer "F.Cu")
-		(at 123.138927 98.642666)
+		(at 123.107858 99.210556)
 		(property "Reference" "G***"
 			(at 0 0 0)
@@
 			(at 0 0 0)
 			(layer "B.SilkS")
+			(hide yes)
 			(effects
 				(font

Commit message: Add files via upload
Parts:
- added FB2: BLM15AX102SN1D, Inductor_SMD:L_0402_1005Metric, F.Cu at (136.4, 72.8)
- added J2: USB_C_Receptacle_PowerOnly_6P, Connector_USB:USB_C_Receptacle_GCT_USB4125-xx-x_6P_TopMnt_Horizontal, F.Cu at (141.2, 76.7)
- added R10: 5.1K, Resistor_SMD:R_0402_1005Metric, F.Cu at (133.6, 77.1)
- added R9: 5.1K, Resistor_SMD:R_0402_1005Metric, F.Cu at (135.8, 78.9)
- added SW3: SW_SPDT, Button_Switch_SMD:SW_SPDT_CK_JS102011SAQN, F.Cu at (120.3, 73.5)
- C7: value C -> 1nF
- moved G*** 2.95 mm to (138.6, 52.2)
Connections:
- J1 pad A4: VBUS -> Net-(SW3-A)
- J1 pad A9: VBUS -> Net-(SW3-A)
- J1 pad B4: VBUS -> Net-(SW3-A)
- J1 pad B9: VBUS -> Net-(SW3-A)
Routing:
- net Net-(SW3-A): track 0.00 -> 39.6 mm
- net VBUS: track 12.8 -> 42.4 mm, vias 0 -> 2
- net /solar_in: track 0.00 -> 19.1 mm
- net Net-(J2-SHIELD): track 0.00 -> 18.2 mm
- net Net-(J2-CC2): track 0.00 -> 6.08 mm, vias 0 -> 2
- net Net-(J2-CC1): track 0.00 -> 4.60 mm, vias 0 -> 2
Other:
- board text added: "Meshing the LoRa V0.0001"
- board text removed: "Meshing the LoRa V0.0001 -alpha"
