File: Lora.kicad_sch (KiCad schematic)
At the start: 49 parts, among them J1 USB_C_Receptacle_USB2.0_16P, SW1 BOOTSEL, SW2 RESET, U1 SX1262IMLTRT, U2 RP2040, U3 W25Q128JVS, U4 AP2112K-3.3, U5 BGS12WN6E6327, Y1 32mhz, Y2 32mhz

Commit message: Add files via upload
Connections:
- net +1V1: now also U2.23 (DVDD), U2.50 (DVDD)
Changed lines of the file:
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@@
+	)
+	(junction
+		(at 228.6 63.5)
+		(diameter 0)
+		(color 0 0 0 0)
 	)
 	(junction
@@
 		)
 		(stroke
+			(width 0)
+			(type default)
+		)
+	)
+	(wire
+		(pts
+			(xy 228.6 63.5) (xy 231.14 63.5)
+		)
+		(stroke

Commit message: dun
Parts:
- AE1: footprint Capacitor_SMD:C_0402_1005Metric -> Connector_PinSocket_2.54mm:PinSocket_1x01_P2.54mm_Vertical
- R7: value 10K -> 5.1K
- U5: value BGS12WN6E6327 -> PE4259; footprint Package_LGA:Infineon_PG-TSNP-6-10_0.7x1.1mm_0.7x1.1mm_P0.4mm -> Package_TO_SOT_SMD:SOT-363_SC-70-6
- Y1: footprint (none) -> Crystal:Crystal_SMD_3225-4Pin_3.2x2.5mm
- Y2: value 32mhz -> 12mhz; footprint (none) -> Crystal:Crystal_SMD_Abracon_ABM8G-4Pin_3.2x2.5mm
Changed lines of the file:
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@@
 			)
 		)
-		(property "Value" "32mhz"
+		(property "Value" "12mhz"
 			(at 359.41 45.212 90)
 			(effects
@@
 			)
 		)
-		(property "Footprint" ""
+		(property "Footprint" "Crystal:Crystal_SMD_Abracon_ABM8G-4Pin_3.2x2.5mm"
 			(at 350.52 40.64 0)
 			(effects
@@
 			)
 		)
-		(property "Value" "BGS12WN6E6327"
+		(property "Value" "PE4259"
 			(at 122.4981 113.03 0)
 			(effects
@@
 			)
 		)
-		(property "Footprint" "Package_LGA:Infineon_PG-TSNP-6-10_0.7x1.1mm_0.7x1.1mm_P0.4mm"
+		(property "Footprint" "Package_TO_SOT_SMD:SOT-363_SC-70-6"
 			(at 119.38 114.3 0)
 			(effects
@@
 			)
 		)
-		(property "Value" "10K"
+		(property "Value" "5.1K"
 			(at 71.12 201.93 90)
 			(effects
@@
 			)
 		)
-		(property "Footprint" "Capacitor_SMD:C_0402_1005Metric"
+		(property "Footprint" "Connector_PinSocket_2.54mm:PinSocket_1x01_P2.54mm_Vertical"
 			(at 177.8 124.46 0)
 			(effects
@@
 			)
 		)
-		(property "Footprint" ""
+		(property "Footprint" "Crystal:Crystal_SMD_3225-4Pin_3.2x2.5mm"
 			(at 91.44 59.69 0)
 			(effects

Commit message: Add files via upload
Parts:
- added FB2: BLM15AX102SN1D, Inductor_SMD:L_0402_1005Metric, symbol Device:FerriteBead_Small
- added J2: USB_C_Receptacle_PowerOnly_6P, Connector_USB:USB_C_Receptacle_GCT_USB4125-xx-x_6P_TopMnt_Horizontal, symbol Connector:USB_C_Receptacle_PowerOnly_6P
- added R10, R9: 5.1K, Resistor_SMD:R_0402_1005Metric, symbol Device:R
- added SW3: SW_SPDT, Button_Switch_SMD:SW_SPDT_CK_JS102011SAQN, symbol Switch:SW_SPDT
- C7: value C -> 1nF
Connections:
- net Earth: now also FB2.2, J2.A12 (GND), J2.B12 (GND), R10.1, R9.2
- net VBUS: now also SW3.2 (B); no longer J1.A4 (VBUS), J1.A9 (VBUS), J1.B4 (VBUS), J1.B9 (VBUS)
- new net: FB2.1, J2.S1 (SHIELD)
- new net: J2.A5 (CC1), R9.1
- new net: J1.A4 (VBUS), J1.A9 (VBUS), J1.B4 (VBUS), J1.B9 (VBUS), SW3.1 (A)
- new net: J2.B5 (CC2), R10.2
- new net solar_in: J2.A9 (VBUS), J2.B9 (VBUS), SW3.3 (C)
